Commit message: add static map goal navigation

File: src/my_robot_description/urdf/my_robot.urdf.xacro (robot description, xacro)
@@ -15,7 +15,4 @@
   <material name="wheel_dark">
     <color rgba="0.03 0.03 0.035 1.0"/>
-  </material>
-  <material name="lidar_black">
-    <color rgba="0.01 0.01 0.01 1.0"/>
   </material>
   <link name="base_footprint"/>
@@ -100,29 +97,4 @@
     <origin xyz="-0.16 0 ${0.026 - base_height / 2.0}" rpy="0 0 0"/>
   </joint>
-  <link name="lidar_link">
-    <visual>
-      <origin xyz="0 0 0" rpy="0 0 0"/>
-      <geometry>
-        <cylinder radius="0.045" length="0.045"/>
-      </geometry>
-      <material name="lidar_black"/>
-    </visual>
-    <collision>
-      <origin xyz="0 0 0" rpy="0 0 0"/>
-      <geometry>
-        <cylinder radius="0.045" length="0.045"/>
-      </geometry>
-    </collision>
-    <inertial>
-      <origin xyz="0 0 0" rpy="0 0 0"/>
-      <mass value="0.2"/>
-      <inertia ixx="0.0001" ixy="0.0" ixz="0.0" iyy="0.0001" iyz="0.0" izz="0.0001"/>
-    </inertial>
-  </link>
-  <joint name="lidar_joint" type="fixed">
-    <parent link="base_link"/>
-    <child link="lidar_link"/>
-    <origin xyz="0.14 0 0.12" rpy="0 0 0"/>
-  </joint>
   <link name="imu_link"/>
   <joint name="imu_joint" type="fixed">
@@ -153,33 +125,4 @@
     </gazebo>
   </xacro:if>
-  <gazebo reference="lidar_link">
-    <sensor name="lidar" type="ray">
-      <always_on>true</always_on>
-      <visualize>true</visualize>
-      <update_rate>10</update_rate>
-      <ray>
-        <scan>
-          <horizontal>
-            <samples>360</samples>
-            <resolution>1</resolution>
-            <min_angle>-3.14159</min_angle>
-            <max_angle>3.14159</max_angle>
-          </horizontal>
-        </scan>
-        <range>
-          <min>0.08</min>
-          <max>8.0</max>
-          <resolution>0.01</resolution>
-        </range>
-      </ray>
-      <plugin name="gazebo_ros_laser" filename="libgazebo_ros_ray_sensor.so">
-        <ros>
-          <remapping>~/out:=scan</remapping>
-        </ros>
-        <output_type>sensor_msgs/LaserScan</output_type>
-        <frame_name>lidar_link</frame_name>
-      </plugin>
-    </sensor>
-  </gazebo>
   <gazebo>
     <plugin name="ground_truth_odom" filename="libgazebo_ros_p3d.so">
